Commit message: new_desgin and no bug

File: new_design/robot_arm1.urdf (robot description, URDF)
Before this commit: robot wx200, 11 links, 10 joints
Links:
- removed link g_bar
- added link gripper_bar, mass 0.030878; collision mesh filename=meshes/gripper_bar.STL; visual mesh filename=meshes/gripper_bar.STL
- link left_gripper: mass 0.010894 -> 0.013875
- link right_gripper: mass 0.010894 -> 0.013875
Joints:
- removed joint g_bar2grlink
- removed joint left_base
- removed joint right_base
- added joint g_par2motor: type fixed, parent ee_arm_link, child gripper_bar, origin xyz=0.004 0 0 rpy=0 0 0, axis 0 0 0
- added joint left_gripper2bar: type prismatic, parent gripper_bar, child left_gripper, origin xyz=0.018 0.054842 0 rpy=0 -1.570796325 1.570796325, axis 0 0 1, limit lower=0 upper=0.03202 effort=5 velocity=1
- added joint right_gripper2bar: type prismatic, parent gripper_bar, child right_gripper, origin xyz=0.018 -0.054991 0 rpy=0 1.570796325 1.570796325, axis 0 0 1, limit lower=0 upper=0.03202 effort=5 velocity=1
- joint ee_gripper: origin xyz=0 -0.06615 0 rpy=0 0 0 -> xyz=0.06615 0 0 rpy=0 0 0; parent g_bar -> gripper_bar
