Commit message: Finished the frameworks.

File: urdf/robot_arm928/robot_arm1.urdf (robot description, URDF)
Before this commit: robot wx200, 11 links, 10 joints
Links:
- link gripper_bar: geometry collision mesh filename=meshes/gripper_bar.STL; visual mesh filename=meshes/gripper_bar.STL
- link left_gripper: geometry collision mesh filename=meshes/left_gripper.STL; visual mesh filename=meshes/left_gripper.STL
- link right_gripper: geometry collision mesh filename=meshes/right_gripper.STL; visual mesh filename=meshes/right_gripper.STL
- link robot_arm: geometry collision mesh filename=meshes/base.stl scale=1 1 1; visual mesh filename=meshes/base.stl scale=1 1 1

Commit message: get_obs

File: urdf/robot_arm928/robot_arm1.urdf (robot description, URDF)
Before this commit: robot wx200, 11 links, 10 joints
Joints:
- joint left_gripper2bar: limit lower=0 upper=0.03202 effort=5 velocity=1 -> lower=0 upper=0.032 effort=5 velocity=1
- joint right_gripper2bar: limit lower=0 upper=0.03202 effort=5 velocity=1 -> lower=0 upper=0.032 effort=5 velocity=1

Commit message: Add files via upload

File: urdf/robot_arm928/robot_arm1.urdf (robot description, URDF)
Before this commit: robot wx200, 11 links, 10 joints
Links:
- link left_gripper: geometry collision mesh filename=meshes/left_finger.STL; visual mesh filename=meshes/left_finger.STL
- link right_gripper: geometry collision mesh filename=meshes/right_finger.STL; visual mesh filename=meshes/right_finger.STL
Joints:
- joint left_gripper2bar: limit lower=0 upper=0.032 effort=5 velocity=1 -> lower=0 upper=0.03202 effort=5 velocity=1; origin xyz=0.018 0.054842 0 rpy=0 0 -3.1416 -> xyz=0.018 0.036991 0 rpy=0 0 -3.1416
- joint right_gripper2bar: limit lower=0 upper=0.032 effort=5 velocity=1 -> lower=0 upper=0.03202 effort=5 velocity=1; origin xyz=0.018 -0.054991 0 rpy=0 0 0 -> xyz=0.018 -0.036991 0 rpy=0 3.1416 0

Commit message: Add files via upload

File: urdf/robot_arm928/robot_arm1.urdf (robot description, URDF)
Before this commit: robot wx200, 11 links, 10 joints
Links:
- link ee_gripper_link: mass 0.001 -> 0
- link left_gripper: geometry collision box size=0.028 0.005 0.02; visual box size=0.028 0.005 0.02
- link right_gripper: geometry collision box size=0.028 0.005 0.02; visual box size=0.028 0.005 0.02
Joints:
- joint left_gripper2bar: limit lower=0 upper=0.03202 effort=5 velocity=1 -> lower=0 upper=0.03202 effort=20 velocity=0.2
- joint right_gripper2bar: limit lower=0 upper=0.03202 effort=5 velocity=1 -> lower=0 upper=0.03202 effort=20 velocity=0.2; mimic (none) -> joint=left_gripper2bar
