Commit message: Add files via upload
update the lego urdf

File: urdf/item_0/0.urdf (robot description, URDF)
Before this commit: robot 2x2, 1 links, 0 joints
Links:
- link base_link: geometry collision box size=0.015 0.015 0.012; visual mesh filename=package://0.STL

File: urdf/item_0/1.urdf (robot description, URDF)
Before this commit: robot 2x2, 1 links, 0 joints
Links:
- link base_link: geometry collision box size=0.015 0.015 0.012; visual mesh filename=package://1.STL

File: urdf/item_0/2.urdf (robot description, URDF)
Before this commit: robot 2x2, 1 links, 0 joints
Links:
- link base_link: geometry collision box size=0.015 0.015 0.012; visual mesh filename=package://2.STL

File: urdf/item_0/3.urdf (robot description, URDF)
Before this commit: robot 2x2, 1 links, 0 joints
Links:
- link base_link: geometry collision box size=0.015 0.015 0.012; visual mesh filename=package://3.STL

File: urdf/item_0/4.urdf (robot description, URDF)
Before this commit: robot 2x2, 1 links, 0 joints
Links:
- link base_link: geometry collision box size=0.015 0.015 0.012; visual mesh filename=package://4.STL

File: urdf/item_0/5.urdf (robot description, URDF)
Before this commit: robot 2x2, 1 links, 0 joints
Links:
- link base_link: geometry collision box size=0.015 0.015 0.012; visual mesh filename=package://5.STL

File: urdf/item_1/0.urdf (robot description, URDF)
Before this commit: robot 2x3, 1 links, 0 joints
Links:
- link base_link: geometry collision box size=0.023 0.015 0.012; visual mesh filename=package://0.STL

File: urdf/item_1/1.urdf (robot description, URDF)
Before this commit: robot 2x3, 1 links, 0 joints
Links:
- link base_link: geometry collision box size=0.023 0.015 0.012; visual mesh filename=package://1.STL

File: urdf/item_1/2.urdf (robot description, URDF)
Before this commit: robot 2x3, 1 links, 0 joints
Links:
- link base_link: geometry collision box size=0.023 0.015 0.012; visual mesh filename=package://2.STL

File: urdf/item_1/3.urdf (robot description, URDF)
Before this commit: robot 2x3, 1 links, 0 joints
Links:
- link base_link: geometry collision box size=0.023 0.015 0.012; visual mesh filename=package://3.STL

File: urdf/item_2/0.urdf (robot description, URDF)
Before this commit: robot 2x4, 1 links, 0 joints
Links:
- link base_link: geometry collision box size=0.033 0.015 0.012; visual mesh filename=package://0.STL

File: urdf/item_2/1.urdf (robot description, URDF)
Before this commit: robot 2x4, 1 links, 0 joints
Links:
- link base_link: geometry collision box size=0.033 0.015 0.012; visual mesh filename=package://1.STL

File: urdf/item_2/2.urdf (robot description, URDF)
Before this commit: robot 2x4, 1 links, 0 joints
Links:
- link base_link: geometry collision box size=0.033 0.015 0.012; visual mesh filename=package://2.STL

File: urdf/item_2/3.urdf (robot description, URDF)
Before this commit: robot 2x4, 1 links, 0 joints
Links:
- link base_link: geometry collision box size=0.033 0.015 0.012; visual mesh filename=package://3.STL

File: urdf/item_2/4.urdf (robot description, URDF)
Before this commit: robot 2x4, 1 links, 0 joints
Links:
- link base_link: geometry collision box size=0.033 0.015 0.012; visual mesh filename=package://4.STL

Commit message: Add files via upload

File: urdf/item_0/0.urdf (robot description, URDF)
Before this commit: robot 2x2, 1 links, 0 joints
Links:
- link base_link: mass 0.0024405 -> 0.01

File: urdf/item_0/1.urdf (robot description, URDF)
Before this commit: robot 2x2, 1 links, 0 joints
Links:
- link base_link: mass 0.0024405 -> 0.01

File: urdf/item_0/2.urdf (robot description, URDF)
Before this commit: robot 2x2, 1 links, 0 joints
Links:
- link base_link: mass 0.0024405 -> 0.01

File: urdf/item_0/3.urdf (robot description, URDF)
Before this commit: robot 2x2, 1 links, 0 joints
Links:
- link base_link: mass 0.0024405 -> 0.01

File: urdf/item_0/4.urdf (robot description, URDF)
Before this commit: robot 2x2, 1 links, 0 joints
Links:
- link base_link: mass 0.0024405 -> 0.01

File: urdf/item_0/5.urdf (robot description, URDF)
Before this commit: robot 2x2, 1 links, 0 joints
Links:
- link base_link: mass 0.0024405 -> 0.01

File: urdf/item_1/0.urdf (robot description, URDF)
Before this commit: robot 2x3, 1 links, 0 joints
Links:
- link base_link: mass 0.0037381 -> 0.01

File: urdf/item_1/1.urdf (robot description, URDF)
Before this commit: robot 2x3, 1 links, 0 joints
Links:
- link base_link: mass 0.0037381 -> 0.01

File: urdf/item_1/2.urdf (robot description, URDF)
Before this commit: robot 2x3, 1 links, 0 joints
Links:
- link base_link: mass 0.0037381 -> 0.01

File: urdf/item_1/3.urdf (robot description, URDF)
Before this commit: robot 2x3, 1 links, 0 joints
Links:
- link base_link: mass 0.0037381 -> 0.01

File: urdf/item_2/0.urdf (robot description, URDF)
Before this commit: robot 2x4, 1 links, 0 joints
Links:
- link base_link: mass 0.0053446 -> 0.01

File: urdf/item_2/1.urdf (robot description, URDF)
Before this commit: robot 2x4, 1 links, 0 joints
Links:
- link base_link: mass 0.0053446 -> 0.01

File: urdf/item_2/2.urdf (robot description, URDF)
Before this commit: robot 2x4, 1 links, 0 joints
Links:
- link base_link: mass 0.0053446 -> 0.01

File: urdf/item_2/3.urdf (robot description, URDF)
Before this commit: robot 2x4, 1 links, 0 joints
Links:
- link base_link: mass 0.0053446 -> 0.01

File: urdf/item_2/4.urdf (robot description, URDF)
Before this commit: robot 2x4, 1 links, 0 joints
Links:
- link base_link: mass 0.0053446 -> 0.01

Commit message: Add files via upload

File: urdf/item_0/0.urdf (robot description, URDF)
Before this commit: robot 2x2, 1 links, 0 joints
Links:
- link base_link: geometry collision box size=0.015 0.015 0.012; visual mesh filename=package://2x2.STL

File: urdf/item_0/1.urdf (robot description, URDF)
Before this commit: robot 2x2, 1 links, 0 joints
Links:
- link base_link: geometry collision box size=0.015 0.015 0.012; visual mesh filename=package://2x2.STL

File: urdf/item_0/2.urdf (robot description, URDF)
Before this commit: robot 2x2, 1 links, 0 joints
Links:
- link base_link: geometry collision box size=0.015 0.015 0.012; visual mesh filename=package://2x2.STL

File: urdf/item_0/3.urdf (robot description, URDF)
Before this commit: robot 2x2, 1 links, 0 joints
Links:
- link base_link: geometry collision box size=0.015 0.015 0.012; visual mesh filename=package://2x2.STL

File: urdf/item_0/4.urdf (robot description, URDF)
Before this commit: robot 2x2, 1 links, 0 joints
Links:
- link base_link: geometry collision box size=0.015 0.015 0.012; visual mesh filename=package://2x2.STL

File: urdf/item_0/5.urdf (robot description, URDF)
Before this commit: robot 2x2, 1 links, 0 joints
Links:
- link base_link: geometry collision box size=0.015 0.015 0.012; visual mesh filename=package://2x2.STL

File: urdf/item_0/6.urdf (robot description, URDF)
Before this commit: robot 2x4, 1 links, 0 joints
Links:
- link base_link: geometry collision box size=0.015 0.015 0.012; visual mesh filename=package://2x2.STL

File: urdf/item_0/7.urdf (robot description, URDF)
Before this commit: robot 2x4, 1 links, 0 joints
Links:
- link base_link: geometry collision box size=0.015 0.015 0.012; visual mesh filename=package://2x2.STL

File: urdf/item_1/0.urdf (robot description, URDF)
Before this commit: robot 2x3, 1 links, 0 joints
Links:
- link base_link: geometry collision box size=0.023 0.015 0.012; visual mesh filename=package://2x3.STL

File: urdf/item_1/1.urdf (robot description, URDF)
Before this commit: robot 2x3, 1 links, 0 joints
Links:
- link base_link: geometry collision box size=0.023 0.015 0.012; visual mesh filename=package://2x3.STL

File: urdf/item_1/2.urdf (robot description, URDF)
Before this commit: robot 2x3, 1 links, 0 joints
Links:
- link base_link: geometry collision box size=0.023 0.015 0.012; visual mesh filename=package://2x3.STL

File: urdf/item_1/3.urdf (robot description, URDF)
Before this commit: robot 2x3, 1 links, 0 joints
Links:
- link base_link: geometry collision box size=0.023 0.015 0.012; visual mesh filename=package://2x3.STL

File: urdf/item_1/4.urdf (robot description, URDF)
Before this commit: robot 2x4, 1 links, 0 joints
Links:
- link base_link: geometry collision box size=0.023 0.015 0.012; visual mesh filename=package://2x3.STL

File: urdf/item_1/5.urdf (robot description, URDF)
Before this commit: robot 2x4, 1 links, 0 joints
Links:
- link base_link: geometry collision box size=0.023 0.015 0.012; visual mesh filename=package://2x3.STL

File: urdf/item_1/6.urdf (robot description, URDF)
Before this commit: robot 2x4, 1 links, 0 joints
Links:
- link base_link: geometry collision box size=0.023 0.015 0.012; visual mesh filename=package://2x3.STL

File: urdf/item_1/7.urdf (robot description, URDF)
Before this commit: robot 2x4, 1 links, 0 joints
Links:
- link base_link: geometry collision box size=0.023 0.015 0.012; visual mesh filename=package://2x3.STL

File: urdf/item_2/0.urdf (robot description, URDF)
Before this commit: robot 2x4, 1 links, 0 joints
Links:
- link base_link: geometry collision box size=0.033 0.015 0.012; visual mesh filename=package://2x4.STL

File: urdf/item_2/1.urdf (robot description, URDF)
Before this commit: robot 2x4, 1 links, 0 joints
Links:
- link base_link: geometry collision box size=0.033 0.015 0.012; visual mesh filename=package://2x4.STL

File: urdf/item_2/2.urdf (robot description, URDF)
Before this commit: robot 2x4, 1 links, 0 joints
Links:
- link base_link: geometry collision box size=0.033 0.015 0.012; visual mesh filename=package://2x4.STL

File: urdf/item_2/3.urdf (robot description, URDF)
Before this commit: robot 2x4, 1 links, 0 joints
Links:
- link base_link: geometry collision box size=0.033 0.015 0.012; visual mesh filename=package://2x4.STL
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
Commit message: zzz_laptop_update

File: urdf/item_0/0.urdf (robot description, URDF)
Before this commit: robot 2x2, 1 links, 0 joints
Links:
- link base_link: geometry collision box size=0.016 0.016 0.012; visual mesh filename=package://2x2.STL

File: urdf/item_0/1.urdf (robot description, URDF)
Before this commit: robot 2x2, 1 links, 0 joints
Links:
- link base_link: geometry collision box size=0.016 0.016 0.012; visual mesh filename=package://2x2.STL

File: urdf/item_0/2.urdf (robot description, URDF)
Before this commit: robot 2x2, 1 links, 0 joints
Links:
- link base_link: geometry collision box size=0.016 0.016 0.012; visual mesh filename=package://2x2.STL

File: urdf/item_0/3.urdf (robot description, URDF)
Before this commit: robot 2x2, 1 links, 0 joints
Links:
- link base_link: geometry collision box size=0.016 0.016 0.012; visual mesh filename=package://2x2.STL

File: urdf/item_0/4.urdf (robot description, URDF)
Before this commit: robot 2x2, 1 links, 0 joints
Links:
- link base_link: geometry collision box size=0.016 0.016 0.012; visual mesh filename=package://2x2.STL

File: urdf/item_0/5.urdf (robot description, URDF)
Before this commit: robot 2x2, 1 links, 0 joints
Links:
- link base_link: geometry collision box size=0.016 0.016 0.012; visual mesh filename=package://2x2.STL

File: urdf/item_0/6.urdf (robot description, URDF)
Before this commit: robot 2x2, 1 links, 0 joints
Links:
- link base_link: geometry collision box size=0.016 0.016 0.012; visual mesh filename=package://2x2.STL

File: urdf/item_0/7.urdf (robot description, URDF)
Before this commit: robot 2x2, 1 links, 0 joints
Links:
- link base_link: geometry collision box size=0.016 0.016 0.012; visual mesh filename=package://2x2.STL

File: urdf/item_1/0.urdf (robot description, URDF)
Before this commit: robot 2x3, 1 links, 0 joints
Links:
- link base_link: geometry collision box size=0.024 0.016 0.012; visual mesh filename=package://2x3.STL

File: urdf/item_1/1.urdf (robot description, URDF)
Before this commit: robot 2x3, 1 links, 0 joints
Links:
- link base_link: geometry collision box size=0.024 0.016 0.012; visual mesh filename=package://2x3.STL

File: urdf/item_1/2.urdf (robot description, URDF)
Before this commit: robot 2x3, 1 links, 0 joints
Links:
- link base_link: geometry collision box size=0.024 0.016 0.012; visual mesh filename=package://2x3.STL

File: urdf/item_1/3.urdf (robot description, URDF)
Before this commit: robot 2x3, 1 links, 0 joints
Links:
- link base_link: geometry collision box size=0.024 0.016 0.012; visual mesh filename=package://2x3.STL

File: urdf/item_1/4.urdf (robot description, URDF)
Before this commit: robot 2x3, 1 links, 0 joints
Links:
- link base_link: geometry collision box size=0.024 0.016 0.012; visual mesh filename=package://2x3.STL

File: urdf/item_1/5.urdf (robot description, URDF)
Before this commit: robot 2x3, 1 links, 0 joints
Links:
- link base_link: geometry collision box size=0.024 0.016 0.012; visual mesh filename=package://2x3.STL

File: urdf/item_1/6.urdf (robot description, URDF)
Before this commit: robot 2x3, 1 links, 0 joints
Links:
- link base_link: geometry collision box size=0.024 0.016 0.012; visual mesh filename=package://2x3.STL

File: urdf/item_1/7.urdf (robot description, URDF)
Before this commit: robot 2x3, 1 links, 0 joints
Links:
- link base_link: geometry collision box size=0.024 0.016 0.012; visual mesh filename=package://2x3.STL

File: urdf/item_2/0.urdf (robot description, URDF)
Before this commit: robot 2x4, 1 links, 0 joints
Links:
- link base_link: geometry collision box size=0.032 0.016 0.012; visual mesh filename=package://2x4.STL

File: urdf/item_2/1.urdf (robot description, URDF)
Before this commit: robot 2x4, 1 links, 0 joints
Links:
- link base_link: geometry collision box size=0.032 0.016 0.012; visual mesh filename=package://2x4.STL

File: urdf/item_2/2.urdf (robot description, URDF)
Before this commit: robot 2x4, 1 links, 0 joints
Links:
- link base_link: geometry collision box size=0.032 0.016 0.012; visual mesh filename=package://2x4.STL

File: urdf/item_2/3.urdf (robot description, URDF)
Before this commit: robot 2x4, 1 links, 0 joints
Links:
- link base_link: geometry collision box size=0.032 0.016 0.012; visual mesh filename=package://2x4.STL
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