Commit message: zzz_laptop_update

File: urdf/box_generator/box_0.urdf (robot description, URDF)
Before this commit: robot 2x2, 1 links, 0 joints
Links:
- link base_link: geometry collision box size=0.045 0.021 0.012; visual box size=0.045 0.021 0.012

File: urdf/box_generator/box_1.urdf (robot description, URDF)
Before this commit: robot 2x2, 1 links, 0 joints
Links:
- link base_link: geometry collision box size=0.021 0.02 0.012; visual box size=0.021 0.02 0.012

File: urdf/box_generator/box_10.urdf (robot description, URDF)
Before this commit: robot 2x2, 1 links, 0 joints
Links:
- link base_link: geometry collision box size=0.024 0.02 0.012; visual box size=0.024 0.02 0.012

File: urdf/box_generator/box_11.urdf (robot description, URDF)
Before this commit: robot 2x2, 1 links, 0 joints
Links:
- link base_link: geometry collision box size=0.018 0.017 0.012; visual box size=0.018 0.017 0.012

File: urdf/box_generator/box_12.urdf (robot description, URDF)
Before this commit: robot 2x2, 1 links, 0 joints
Links:
- link base_link: geometry collision box size=0.023 0.017 0.012; visual box size=0.023 0.017 0.012

File: urdf/box_generator/box_13.urdf (robot description, URDF)
Before this commit: robot 2x2, 1 links, 0 joints
Links:
- link base_link: geometry collision box size=0.038 0.02 0.012; visual box size=0.038 0.02 0.012

File: urdf/box_generator/box_14.urdf (robot description, URDF)
Before this commit: robot 2x2, 1 links, 0 joints
Links:
- link base_link: geometry collision box size=0.035 0.02 0.012; visual box size=0.035 0.02 0.012

File: urdf/box_generator/box_15.urdf (robot description, URDF)
Before this commit: robot 2x2, 1 links, 0 joints
Links:
- link base_link: geometry collision box size=0.037 0.018 0.012; visual box size=0.037 0.018 0.012

File: urdf/box_generator/box_16.urdf (robot description, URDF)
Before this commit: robot 2x2, 1 links, 0 joints
Links:
- link base_link: geometry collision box size=0.04 0.035 0.012; visual box size=0.04 0.035 0.012

File: urdf/box_generator/box_17.urdf (robot description, URDF)
Before this commit: robot 2x2, 1 links, 0 joints
Links:
- link base_link: geometry collision box size=0.039 0.029 0.012; visual box size=0.039 0.029 0.012

File: urdf/box_generator/box_18.urdf (robot description, URDF)
Before this commit: robot 2x2, 1 links, 0 joints
Links:
- link base_link: geometry collision box size=0.048 0.032 0.012; visual box size=0.048 0.032 0.012

File: urdf/box_generator/box_19.urdf (robot description, URDF)
Before this commit: robot 2x2, 1 links, 0 joints
Links:
- link base_link: geometry collision box size=0.037 0.02 0.012; visual box size=0.037 0.02 0.012

File: urdf/box_generator/box_2.urdf (robot description, URDF)
Before this commit: robot 2x2, 1 links, 0 joints
Links:
- link base_link: geometry collision box size=0.024 0.018 0.012; visual box size=0.024 0.018 0.012

File: urdf/box_generator/box_20.urdf (robot description, URDF)
Before this commit: robot 2x2, 1 links, 0 joints
Links:
- link base_link: geometry collision box size=0.038 0.03 0.012; visual box size=0.038 0.03 0.012

File: urdf/box_generator/box_21.urdf (robot description, URDF)
Before this commit: robot 2x2, 1 links, 0 joints
Links:
- link base_link: geometry collision box size=0.018 0.017 0.012; visual box size=0.018 0.017 0.012

File: urdf/box_generator/box_22.urdf (robot description, URDF)
Before this commit: robot 2x2, 1 links, 0 joints
Links:
- link base_link: geometry collision box size=0.033 0.018 0.012; visual box size=0.033 0.018 0.012

File: urdf/box_generator/box_23.urdf (robot description, URDF)
Before this commit: robot 2x2, 1 links, 0 joints
Links:
- link base_link: geometry collision box size=0.017 0.017 0.012; visual box size=0.017 0.017 0.012

File: urdf/box_generator/box_24.urdf (robot description, URDF)
Before this commit: robot 2x2, 1 links, 0 joints
Links:
- link base_link: geometry collision box size=0.021 0.017 0.012; visual box size=0.021 0.017 0.012

File: urdf/box_generator/box_25.urdf (robot description, URDF)
Before this commit: robot 2x2, 1 links, 0 joints
Links:
- link base_link: geometry collision box size=0.017 0.017 0.012; visual box size=0.017 0.017 0.012

File: urdf/box_generator/box_26.urdf (robot description, URDF)
Before this commit: robot 2x2, 1 links, 0 joints
Links:
- link base_link: geometry collision box size=0.017 0.017 0.012; visual box size=0.017 0.017 0.012
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