Commit message: zzz_laptop_update

File: urdf/plane_1.urdf (robot description, URDF)
Before this commit: robot plane, 1 links, 0 joints
Links:
- link planeLink: geometry collision box size=1 1 10; visual mesh filename=plane100.obj scale=0.201 0.201 1

Commit message: zzz lab update

File: urdf/plane_1.urdf (robot description, URDF)
Before this commit: robot plane, 1 links, 0 joints
Links:
- link planeLink: geometry collision box size=1 1 10; visual mesh filename=plane100.obj scale=0.221 0.221 1

Commit message: zzz_laptop_update

File: urdf/plane_1.urdf (robot description, URDF)
Before this commit: robot plane, 1 links, 0 joints
Links:
- link planeLink: geometry collision box size=10 10 10; visual mesh filename=plane100.obj scale=0.221 0.221 1
