Commit message: zzz_laptop_update

File: urdf/box_generator/generation_1/box_0.urdf (robot description, URDF)
Before this commit: robot 2x2, 1 links, 0 joints
Links:
- link base_link: geometry collision box size=0.045 0.034 0.012; visual box size=0.045 0.034 0.012

File: urdf/box_generator/generation_1/box_1.urdf (robot description, URDF)
Before this commit: robot 2x2, 1 links, 0 joints
Links:
- link base_link: geometry collision box size=0.04 0.024 0.015; visual box size=0.04 0.024 0.015

File: urdf/box_generator/generation_1/box_10.urdf (robot description, URDF)
Before this commit: robot 2x2, 1 links, 0 joints
Links:
- link base_link: geometry collision box size=0.023 0.021 0.019; visual box size=0.023 0.021 0.019

File: urdf/box_generator/generation_1/box_11.urdf (robot description, URDF)
Before this commit: robot 2x2, 1 links, 0 joints
Links:
- link base_link: geometry collision box size=0.022 0.02 0.012; visual box size=0.022 0.02 0.012

File: urdf/box_generator/generation_1/box_12.urdf (robot description, URDF)
Before this commit: robot 2x2, 1 links, 0 joints
Links:
- link base_link: geometry collision box size=0.032 0.027 0.017; visual box size=0.032 0.027 0.017

File: urdf/box_generator/generation_1/box_13.urdf (robot description, URDF)
Before this commit: robot 2x2, 1 links, 0 joints
Links:
- link base_link: geometry collision box size=0.021 0.016 0.013; visual box size=0.021 0.016 0.013

File: urdf/box_generator/generation_1/box_14.urdf (robot description, URDF)
Before this commit: robot 2x2, 1 links, 0 joints
Links:
- link base_link: geometry collision box size=0.04 0.02 0.013; visual box size=0.04 0.02 0.013

File: urdf/box_generator/generation_1/box_15.urdf (robot description, URDF)
Before this commit: robot 2x2, 1 links, 0 joints
Links:
- link base_link: geometry collision box size=0.025 0.02 0.014; visual box size=0.025 0.02 0.014

File: urdf/box_generator/generation_1/box_16.urdf (robot description, URDF)
Before this commit: robot 2x2, 1 links, 0 joints
Links:
- link base_link: geometry collision box size=0.027 0.024 0.014; visual box size=0.027 0.024 0.014

File: urdf/box_generator/generation_1/box_17.urdf (robot description, URDF)
Before this commit: robot 2x2, 1 links, 0 joints
Links:
- link base_link: geometry collision box size=0.043 0.026 0.017; visual box size=0.043 0.026 0.017

File: urdf/box_generator/generation_1/box_18.urdf (robot description, URDF)
Before this commit: robot 2x2, 1 links, 0 joints
Links:
- link base_link: geometry collision box size=0.029 0.028 0.018; visual box size=0.029 0.028 0.018

File: urdf/box_generator/generation_1/box_19.urdf (robot description, URDF)
Before this commit: robot 2x2, 1 links, 0 joints
Links:
- link base_link: geometry collision box size=0.046 0.029 0.018; visual box size=0.046 0.029 0.018

File: urdf/box_generator/generation_1/box_2.urdf (robot description, URDF)
Before this commit: robot 2x2, 1 links, 0 joints
Links:
- link base_link: geometry collision box size=0.02 0.019 0.015; visual box size=0.02 0.019 0.015

File: urdf/box_generator/generation_1/box_20.urdf (robot description, URDF)
Before this commit: robot 2x2, 1 links, 0 joints
Links:
- link base_link: geometry collision box size=0.019 0.016 0.019; visual box size=0.019 0.016 0.019

File: urdf/box_generator/generation_1/box_21.urdf (robot description, URDF)
Before this commit: robot 2x2, 1 links, 0 joints
Links:
- link base_link: geometry collision box size=0.04 0.033 0.014; visual box size=0.04 0.033 0.014

File: urdf/box_generator/generation_1/box_22.urdf (robot description, URDF)
Before this commit: robot 2x2, 1 links, 0 joints
Links:
- link base_link: geometry collision box size=0.04 0.033 0.015; visual box size=0.04 0.033 0.015

File: urdf/box_generator/generation_1/box_23.urdf (robot description, URDF)
Before this commit: robot 2x2, 1 links, 0 joints
Links:
- link base_link: geometry collision box size=0.027 0.024 0.011; visual box size=0.027 0.024 0.011

File: urdf/box_generator/generation_1/box_24.urdf (robot description, URDF)
Before this commit: robot 2x2, 1 links, 0 joints
Links:
- link base_link: geometry collision box size=0.039 0.02 0.011; visual box size=0.039 0.02 0.011

File: urdf/box_generator/generation_1/box_25.urdf (robot description, URDF)
Before this commit: robot 2x2, 1 links, 0 joints
Links:
- link base_link: geometry collision box size=0.045 0.016 0.013; visual box size=0.045 0.016 0.013

File: urdf/box_generator/generation_1/box_26.urdf (robot description, URDF)
Before this commit: robot 2x2, 1 links, 0 joints
Links:
- link base_link: geometry collision box size=0.047 0.022 0.019; visual box size=0.047 0.022 0.019
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