Commit message: zzz_laptop_update

File: urdf/box_generator/yolo_random_thread_0/box_0.urdf (robot description, URDF)
Before this commit: robot 2x2, 1 links, 0 joints
Links:
- link base_link: geometry collision box size=0.018 0.018 0.012; visual box size=0.018 0.018 0.012

File: urdf/box_generator/yolo_random_thread_0/box_1.urdf (robot description, URDF)
Before this commit: robot 2x2, 1 links, 0 joints
Links:
- link base_link: geometry collision box size=0.031 0.031 0.012; visual box size=0.031 0.031 0.012

File: urdf/box_generator/yolo_random_thread_0/box_2.urdf (robot description, URDF)
Before this commit: robot 2x2, 1 links, 0 joints
Links:
- link base_link: geometry collision box size=0.028 0.02 0.012; visual box size=0.028 0.02 0.012

File: urdf/box_generator/yolo_random_thread_0/box_3.urdf (robot description, URDF)
Before this commit: robot 2x2, 1 links, 0 joints
Links:
- link base_link: geometry collision box size=0.035 0.031 0.012; visual box size=0.035 0.031 0.012

File: urdf/box_generator/yolo_random_thread_0/box_4.urdf (robot description, URDF)
Before this commit: robot 2x2, 1 links, 0 joints
Links:
- link base_link: geometry collision box size=0.033 0.032 0.012; visual box size=0.033 0.032 0.012

File: urdf/box_generator/yolo_random_thread_1/box_1.urdf (robot description, URDF)
Before this commit: robot 2x2, 1 links, 0 joints
Links:
- link base_link: geometry collision box size=0.025 0.02 0.012; visual box size=0.025 0.02 0.012

File: urdf/box_generator/yolo_random_thread_1/box_2.urdf (robot description, URDF)
Before this commit: robot 2x2, 1 links, 0 joints
Links:
- link base_link: geometry collision box size=0.017 0.017 0.012; visual box size=0.017 0.017 0.012

File: urdf/box_generator/yolo_random_thread_1/box_3.urdf (robot description, URDF)
Before this commit: robot 2x2, 1 links, 0 joints
Links:
- link base_link: geometry collision box size=0.04 0.024 0.012; visual box size=0.04 0.024 0.012

File: urdf/box_generator/yolo_random_thread_1/box_4.urdf (robot description, URDF)
Before this commit: robot 2x2, 1 links, 0 joints
Links:
- link base_link: geometry collision box size=0.034 0.032 0.012; visual box size=0.034 0.032 0.012

File: urdf/box_generator/yolo_random_thread_1/box_5.urdf (robot description, URDF)
Before this commit: robot 2x2, 1 links, 0 joints
Links:
- link base_link: geometry collision box size=0.017 0.017 0.012; visual box size=0.017 0.017 0.012

File: urdf/box_generator/yolo_random_thread_1/box_6.urdf (robot description, URDF)
Before this commit: robot 2x2, 1 links, 0 joints
Links:
- link base_link: geometry collision box size=0.02 0.018 0.012; visual box size=0.02 0.018 0.012

File: urdf/box_generator/yolo_random_thread_1/box_7.urdf (robot description, URDF)
Before this commit: robot 2x2, 1 links, 0 joints
Links:
- link base_link: geometry collision box size=0.035 0.025 0.012; visual box size=0.035 0.025 0.012

File: urdf/box_generator/yolo_random_thread_1/box_8.urdf (robot description, URDF)
Before this commit: robot 2x2, 1 links, 0 joints
Links:
- link base_link: geometry collision box size=0.027 0.018 0.012; visual box size=0.027 0.018 0.012

File: urdf/box_generator/yolo_random_thread_1/box_9.urdf (robot description, URDF)
Before this commit: robot 2x2, 1 links, 0 joints
Links:
- link base_link: geometry collision box size=0.046 0.02 0.012; visual box size=0.046 0.02 0.012

File: urdf/box_generator/yolo_random_thread_2/box_0.urdf (robot description, URDF)
Before this commit: robot 2x2, 1 links, 0 joints
Links:
- link base_link: geometry collision box size=0.04 0.018 0.012; visual box size=0.04 0.018 0.012

File: urdf/box_generator/yolo_random_thread_2/box_1.urdf (robot description, URDF)
Before this commit: robot 2x2, 1 links, 0 joints
Links:
- link base_link: geometry collision box size=0.038 0.035 0.012; visual box size=0.038 0.035 0.012

File: urdf/box_generator/yolo_random_thread_2/box_2.urdf (robot description, URDF)
Before this commit: robot 2x2, 1 links, 0 joints
Links:
- link base_link: geometry collision box size=0.018 0.017 0.012; visual box size=0.018 0.017 0.012

File: urdf/box_generator/yolo_random_thread_2/box_3.urdf (robot description, URDF)
Before this commit: robot 2x2, 1 links, 0 joints
Links:
- link base_link: geometry collision box size=0.043 0.021 0.012; visual box size=0.043 0.021 0.012

File: urdf/box_generator/yolo_random_thread_2/box_7.urdf (robot description, URDF)
Before this commit: robot 2x2, 1 links, 0 joints
Links:
- link base_link: geometry collision box size=0.024 0.023 0.012; visual box size=0.024 0.023 0.012

File: urdf/box_generator/yolo_random_thread_2/box_8.urdf (robot description, URDF)
Before this commit: robot 2x2, 1 links, 0 joints
Links:
- link base_link: geometry collision box size=0.039 0.032 0.012; visual box size=0.039 0.032 0.012
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