Commit message: zzz_laptop_update

File: real_world_data_demo/cfg_4_520/urdf/num_10/img_4/lego_demo_3.urdf (robot description, URDF)
Before this commit: robot 2x2, 1 links, 0 joints
Links:
- link base_link: geometry collision box size=0.022 0.02 0.012; visual box size=0.022 0.02 0.012

File: real_world_data_demo/cfg_4_520/urdf/num_10/img_4/lego_demo_8.urdf (robot description, URDF)
Before this commit: robot 2x2, 1 links, 0 joints
Links:
- link base_link: geometry collision box size=0.032 0.016 0.012; visual box size=0.032 0.016 0.012

File: urdf/knolling_box/knolling_box_0.urdf (robot description, URDF)
Before this commit: robot 2x2, 1 links, 0 joints
Links:
- link base_link: geometry collision box size=0.0332 0.0272 0.012; visual box size=0.0332 0.0272 0.012

File: urdf/knolling_box/knolling_box_1.urdf (robot description, URDF)
Before this commit: robot 2x2, 1 links, 0 joints
Links:
- link base_link: geometry collision box size=0.0313 0.0169 0.012; visual box size=0.0313 0.0169 0.012

File: urdf/knolling_box/knolling_box_2.urdf (robot description, URDF)
Before this commit: robot 2x2, 1 links, 0 joints
Links:
- link base_link: geometry collision box size=0.03 0.0151 0.012; visual box size=0.03 0.0151 0.012

File: urdf/knolling_box/knolling_box_3.urdf (robot description, URDF)
Before this commit: robot 2x2, 1 links, 0 joints
Links:
- link base_link: geometry collision box size=0.0298 0.0168 0.012; visual box size=0.0298 0.0168 0.012

File: urdf/knolling_box/knolling_box_4.urdf (robot description, URDF)
Before this commit: robot 2x2, 1 links, 0 joints
Links:
- link base_link: geometry collision box size=0.0259 0.0142 0.012; visual box size=0.0259 0.0142 0.012

File: urdf/knolling_box/knolling_box_5.urdf (robot description, URDF)
Before this commit: robot 2x2, 1 links, 0 joints
Links:
- link base_link: geometry collision box size=0.0279 0.0257 0.012; visual box size=0.0279 0.0257 0.012

File: urdf/knolling_box/knolling_box_6.urdf (robot description, URDF)
Before this commit: robot 2x2, 1 links, 0 joints
Links:
- link base_link: geometry collision box size=0.0211 0.0209 0.012; visual box size=0.0211 0.0209 0.012

File: urdf/knolling_box/knolling_box_7.urdf (robot description, URDF)
Before this commit: robot 2x2, 1 links, 0 joints
Links:
- link base_link: geometry collision box size=0.0457 0.0172 0.012; visual box size=0.0457 0.0172 0.012

File: urdf/knolling_box/knolling_box_8.urdf (robot description, URDF)
Before this commit: robot 2x2, 1 links, 0 joints
Links:
- link base_link: geometry collision box size=0.0188 0.0176 0.012; visual box size=0.0188 0.0176 0.012

File: urdf/knolling_box/knolling_box_9.urdf (robot description, URDF)
Before this commit: robot 2x2, 1 links, 0 joints
Links:
- link base_link: geometry collision box size=0.0247 0.0173 0.012; visual box size=0.0247 0.0173 0.012
