Commit message: zzz_laptop_update

File: urdf/knolling_box/knolling_box_0.urdf (robot description, URDF)
Before this commit: robot 2x2, 1 links, 0 joints
Links:
- link base_link: geometry collision box size=0.020833 0.014583 0.012; visual box size=0.020833 0.014583 0.012

File: urdf/knolling_box/knolling_box_1.urdf (robot description, URDF)
Before this commit: robot 2x2, 1 links, 0 joints
Links:
- link base_link: geometry collision box size=0.029167 0.015278 0.012; visual box size=0.029167 0.015278 0.012

File: urdf/knolling_box/knolling_box_2.urdf (robot description, URDF)
Before this commit: robot 2x2, 1 links, 0 joints
Links:
- link base_link: geometry collision box size=0.028125 0.015278 0.012; visual box size=0.028125 0.015278 0.012

File: urdf/knolling_box/knolling_box_3.urdf (robot description, URDF)
Before this commit: robot 2x2, 1 links, 0 joints
Links:
- link base_link: geometry collision box size=0.029687 0.015278 0.012; visual box size=0.029687 0.015278 0.012

Commit message: zzz_laptop_update

File: urdf/knolling_box/knolling_box_0.urdf (robot description, URDF)
Before this commit: robot 2x2, 1 links, 0 joints
Links:
- link base_link: geometry collision box size=0.021354 0.015278 0.012; visual box size=0.021354 0.015278 0.012

File: urdf/knolling_box/knolling_box_1.urdf (robot description, URDF)
Before this commit: robot 2x2, 1 links, 0 joints
Links:
- link base_link: geometry collision box size=0.028646 0.014583 0.012; visual box size=0.028646 0.014583 0.012

File: urdf/knolling_box/knolling_box_3.urdf (robot description, URDF)
Before this commit: robot 2x2, 1 links, 0 joints
Links:
- link base_link: geometry collision box size=0.029167 0.015278 0.012; visual box size=0.029167 0.015278 0.012

Commit message: zzz_laptop_update

File: urdf/knolling_box/knolling_box_0.urdf (robot description, URDF)
Before this commit: robot 2x2, 1 links, 0 joints
Links:
- link base_link: geometry collision box size=0.012074 0.010706 0.012; visual box size=0.012074 0.010706 0.012

File: urdf/knolling_box/knolling_box_1.urdf (robot description, URDF)
Before this commit: robot 2x2, 1 links, 0 joints
Links:
- link base_link: geometry collision box size=0.012068 0.0092366 0.012; visual box size=0.012068 0.0092366 0.012

File: urdf/knolling_box/knolling_box_2.urdf (robot description, URDF)
Before this commit: robot 2x2, 1 links, 0 joints
Links:
- link base_link: geometry collision box size=0.050725 0.049375 0.012; visual box size=0.050725 0.049375 0.012

File: urdf/knolling_box/knolling_box_3.urdf (robot description, URDF)
Before this commit: robot 2x2, 1 links, 0 joints
Links:
- link base_link: geometry collision box size=0.027858 0.015763 0.012; visual box size=0.027858 0.015763 0.012

File: urdf/knolling_box/knolling_box_4.urdf (robot description, URDF)
Before this commit: robot 2x2, 1 links, 0 joints
Links:
- link base_link: geometry collision box size=0.013579 0.012033 0.012; visual box size=0.013579 0.012033 0.012

Commit message: zzz_laptop_update

File: urdf/knolling_box/knolling_box_0.urdf (robot description, URDF)
Before this commit: robot 2x2, 1 links, 0 joints
Links:
- link base_link: geometry collision box size=0.016 0.015 0.012; visual box size=0.016 0.015 0.012

File: urdf/knolling_box/knolling_box_1.urdf (robot description, URDF)
Before this commit: robot 2x2, 1 links, 0 joints
Links:
- link base_link: geometry collision box size=0.015 0.015 0.012; visual box size=0.015 0.015 0.012

File: urdf/knolling_box/knolling_box_2.urdf (robot description, URDF)
Before this commit: robot 2x2, 1 links, 0 joints
Links:
- link base_link: geometry collision box size=0.015 0.014 0.012; visual box size=0.015 0.014 0.012

File: urdf/knolling_box/knolling_box_3.urdf (robot description, URDF)
Before this commit: robot 2x2, 1 links, 0 joints
Links:
- link base_link: geometry collision box size=0.024 0.015 0.012; visual box size=0.024 0.015 0.012

File: urdf/knolling_box/knolling_box_4.urdf (robot description, URDF)
Before this commit: robot 2x2, 1 links, 0 joints
Links:
- link base_link: geometry collision box size=0.031 0.015 0.012; visual box size=0.031 0.015 0.012

File: urdf/plane_1.urdf (robot description, URDF)
Before this commit: robot plane, 1 links, 0 joints
Links:
- link planeLink: geometry collision box size=10 10 10; visual mesh filename=plane100.obj scale=0.2 0.2 1

Commit message: zzz_laptop_update

File: urdf/knolling_box/knolling_box_0.urdf (robot description, URDF)
Before this commit: robot 2x2, 1 links, 0 joints
Links:
- link base_link: geometry collision box size=0.03 0.023 0.012; visual box size=0.03 0.023 0.012

File: urdf/knolling_box/knolling_box_1.urdf (robot description, URDF)
Before this commit: robot 2x2, 1 links, 0 joints
Links:
- link base_link: geometry collision box size=0.02 0.017 0.012; visual box size=0.02 0.017 0.012

File: urdf/knolling_box/knolling_box_2.urdf (robot description, URDF)
Before this commit: robot 2x2, 1 links, 0 joints
Links:
- link base_link: geometry collision box size=0.021 0.019 0.012; visual box size=0.021 0.019 0.012

File: urdf/knolling_box/knolling_box_3.urdf (robot description, URDF)
Before this commit: robot 2x2, 1 links, 0 joints
Links:
- link base_link: geometry collision box size=0.021 0.021 0.012; visual box size=0.021 0.021 0.012

File: urdf/knolling_box/knolling_box_4.urdf (robot description, URDF)
Before this commit: robot 2x2, 1 links, 0 joints
Links:
- link base_link: geometry collision box size=0.015 0.014 0.012; visual box size=0.015 0.014 0.012

File: urdf/knolling_box/knolling_box_5.urdf (robot description, URDF)
Before this commit: robot 2x2, 1 links, 0 joints
Links:
- link base_link: geometry collision box size=0.018 0.014 0.012; visual box size=0.018 0.014 0.012

File: urdf/knolling_box/knolling_box_6.urdf (robot description, URDF)
Before this commit: robot 2x2, 1 links, 0 joints
Links:
- link base_link: geometry collision box size=0.016 0.015 0.012; visual box size=0.016 0.015 0.012

File: urdf/knolling_box/knolling_box_7.urdf (robot description, URDF)
Before this commit: robot 2x2, 1 links, 0 joints
Links:
- link base_link: geometry collision box size=0.031 0.022 0.012; visual box size=0.031 0.022 0.012

File: urdf/knolling_box/knolling_box_8.urdf (robot description, URDF)
Before this commit: robot 2x2, 1 links, 0 joints
Links:
- link base_link: geometry collision box size=0.029 0.018 0.012; visual box size=0.029 0.018 0.012

File: urdf/knolling_box/knolling_box_9.urdf (robot description, URDF)
Before this commit: robot 2x2, 1 links, 0 joints
Links:
- link base_link: geometry collision box size=0.018 0.015 0.012; visual box size=0.018 0.015 0.012

Commit message: zzz_laptop_update

File: urdf/knolling_box/knolling_box_0.urdf (robot description, URDF)
Before this commit: robot 2x2, 1 links, 0 joints
Links:
- link base_link: geometry collision box size=0.033 0.02 0.012; visual box size=0.033 0.02 0.012

File: urdf/knolling_box/knolling_box_1.urdf (robot description, URDF)
Before this commit: robot 2x2, 1 links, 0 joints
Links:
- link base_link: geometry collision box size=0.03 0.02 0.012; visual box size=0.03 0.02 0.012

File: urdf/knolling_box/knolling_box_2.urdf (robot description, URDF)
Before this commit: robot 2x2, 1 links, 0 joints
Links:
- link base_link: geometry collision box size=0.046 0.03 0.012; visual box size=0.046 0.03 0.012

File: urdf/knolling_box/knolling_box_3.urdf (robot description, URDF)
Before this commit: robot 2x2, 1 links, 0 joints
Links:
- link base_link: geometry collision box size=0.022 0.02 0.012; visual box size=0.022 0.02 0.012

File: urdf/knolling_box/knolling_box_4.urdf (robot description, URDF)
Before this commit: robot 2x2, 1 links, 0 joints
Links:
- link base_link: geometry collision box size=0.041 0.018 0.012; visual box size=0.041 0.018 0.012

File: urdf/knolling_box/knolling_box_5.urdf (robot description, URDF)
Before this commit: robot 2x2, 1 links, 0 joints
Links:
- link base_link: geometry collision box size=0.036 0.03 0.012; visual box size=0.036 0.03 0.012

File: urdf/knolling_box/knolling_box_6.urdf (robot description, URDF)
Before this commit: robot 2x2, 1 links, 0 joints
Links:
- link base_link: geometry collision box size=0.037 0.029 0.012; visual box size=0.037 0.029 0.012

File: urdf/knolling_box/knolling_box_7.urdf (robot description, URDF)
Before this commit: robot 2x2, 1 links, 0 joints
Links:
- link base_link: geometry collision box size=0.03 0.018 0.012; visual box size=0.03 0.018 0.012

File: urdf/knolling_box/knolling_box_8.urdf (robot description, URDF)
Before this commit: robot 2x2, 1 links, 0 joints
Links:
- link base_link: geometry collision box size=0.022 0.021 0.012; visual box size=0.022 0.021 0.012

File: urdf/knolling_box/knolling_box_9.urdf (robot description, URDF)
Before this commit: robot 2x2, 1 links, 0 joints
Links:
- link base_link: geometry collision box size=0.045 0.02 0.012; visual box size=0.045 0.02 0.012

Commit message: zzz_laptop_update

File: urdf/knolling_box/knolling_box_0.urdf (robot description, URDF)
Before this commit: robot 2x2, 1 links, 0 joints
Links:
- link base_link: geometry collision box size=0.0307 0.0166 0.012; visual box size=0.0307 0.0166 0.012

File: urdf/knolling_box/knolling_box_1.urdf (robot description, URDF)
Before this commit: robot 2x2, 1 links, 0 joints
Links:
- link base_link: geometry collision box size=0.021 0.0187 0.012; visual box size=0.021 0.0187 0.012

File: urdf/knolling_box/knolling_box_2.urdf (robot description, URDF)
Before this commit: robot 2x2, 1 links, 0 joints
Links:
- link base_link: geometry collision box size=0.0289 0.026 0.012; visual box size=0.0289 0.026 0.012

File: urdf/knolling_box/knolling_box_3.urdf (robot description, URDF)
Before this commit: robot 2x2, 1 links, 0 joints
Links:
- link base_link: geometry collision box size=0.0199 0.0192 0.012; visual box size=0.0199 0.0192 0.012

File: urdf/knolling_box/knolling_box_4.urdf (robot description, URDF)
Before this commit: robot 2x2, 1 links, 0 joints
Links:
- link base_link: geometry collision box size=0.0212 0.0157 0.012; visual box size=0.0212 0.0157 0.012

File: urdf/knolling_box/knolling_box_5.urdf (robot description, URDF)
Before this commit: robot 2x2, 1 links, 0 joints
Links:
- link base_link: geometry collision box size=0.0319 0.0233 0.012; visual box size=0.0319 0.0233 0.012

File: urdf/knolling_box/knolling_box_6.urdf (robot description, URDF)
Before this commit: robot 2x2, 1 links, 0 joints
Links:
- link base_link: geometry collision box size=0.0439 0.0186 0.012; visual box size=0.0439 0.0186 0.012

File: urdf/knolling_box/knolling_box_7.urdf (robot description, URDF)
Before this commit: robot 2x2, 1 links, 0 joints
Links:
- link base_link: geometry collision box size=0.022 0.0186 0.012; visual box size=0.022 0.0186 0.012

File: urdf/knolling_box/knolling_box_8.urdf (robot description, URDF)
Before this commit: robot 2x2, 1 links, 0 joints
Links:
- link base_link: geometry collision box size=0.0212 0.0206 0.012; visual box size=0.0212 0.0206 0.012

File: urdf/knolling_box/knolling_box_9.urdf (robot description, URDF)
Before this commit: robot 2x2, 1 links, 0 joints
Links:
- link base_link: geometry collision box size=0.0312 0.016 0.012; visual box size=0.0312 0.016 0.012

Commit message: zzz_laptop_update

File: urdf/knolling_box/knolling_box_0.urdf (robot description, URDF)
Before this commit: robot 2x2, 1 links, 0 joints
Links:
- link base_link: geometry collision box size=0.0293 0.0172 0.012; visual box size=0.0293 0.0172 0.012

File: urdf/knolling_box/knolling_box_1.urdf (robot description, URDF)
Before this commit: robot 2x2, 1 links, 0 joints
Links:
- link base_link: geometry collision box size=0.0163 0.0078 0.012; visual box size=0.0163 0.0078 0.012
