Commit message: zzz_laptop_update

File: urdf/knolling_box/box_0.urdf (robot description, URDF)
Before this commit: robot 2x2, 1 links, 0 joints
Links:
- link base_link: geometry collision box size=0.0311 0.0294 0.012; visual box size=0.0311 0.0294 0.012

File: urdf/knolling_box/box_1.urdf (robot description, URDF)
Before this commit: robot 2x2, 1 links, 0 joints
Links:
- link base_link: geometry collision box size=0.0319 0.015 0.012; visual box size=0.0319 0.015 0.012

File: urdf/knolling_box/box_10.urdf (robot description, URDF)
Before this commit: robot 2x2, 1 links, 0 joints
Links:
- link base_link: geometry collision box size=0.029688 0.024171 0.012; visual box size=0.029688 0.024171 0.012

File: urdf/knolling_box/box_2.urdf (robot description, URDF)
Before this commit: robot 2x2, 1 links, 0 joints
Links:
- link base_link: geometry collision box size=0.0279 0.0227 0.012; visual box size=0.0279 0.0227 0.012

File: urdf/knolling_box/box_3.urdf (robot description, URDF)
Before this commit: robot 2x2, 1 links, 0 joints
Links:
- link base_link: geometry collision box size=0.0345 0.0248 0.012; visual box size=0.0345 0.0248 0.012

File: urdf/knolling_box/box_4.urdf (robot description, URDF)
Before this commit: robot 2x2, 1 links, 0 joints
Links:
- link base_link: geometry collision box size=0.0454 0.0192 0.012; visual box size=0.0454 0.0192 0.012

File: urdf/knolling_box/box_5.urdf (robot description, URDF)
Before this commit: robot 2x2, 1 links, 0 joints
Links:
- link base_link: geometry collision box size=0.0295 0.0199 0.012; visual box size=0.0295 0.0199 0.012

File: urdf/knolling_box/box_6.urdf (robot description, URDF)
Before this commit: robot 2x2, 1 links, 0 joints
Links:
- link base_link: geometry collision box size=0.0331 0.0183 0.012; visual box size=0.0331 0.0183 0.012

File: urdf/knolling_box/box_7.urdf (robot description, URDF)
Before this commit: robot 2x2, 1 links, 0 joints
Links:
- link base_link: geometry collision box size=0.0266 0.0169 0.012; visual box size=0.0266 0.0169 0.012

File: urdf/knolling_box/box_8.urdf (robot description, URDF)
Before this commit: robot 2x2, 1 links, 0 joints
Links:
- link base_link: geometry collision box size=0.0309 0.0266 0.012; visual box size=0.0309 0.0266 0.012

File: urdf/knolling_box/box_9.urdf (robot description, URDF)
Before this commit: robot 2x2, 1 links, 0 joints
Links:
- link base_link: geometry collision box size=0.0442 0.0302 0.012; visual box size=0.0442 0.0302 0.012

Commit message: zzz xps update

File: urdf/knolling_box/box_0.urdf (robot description, URDF)
Before this commit: robot 2x2, 1 links, 0 joints
Links:
- link base_link: geometry collision box size=0.017 0.026 0.012; visual box size=0.017 0.026 0.012

File: urdf/knolling_box/box_1.urdf (robot description, URDF)
Before this commit: robot 2x2, 1 links, 0 joints
Links:
- link base_link: geometry collision box size=0.023 0.024 0.012; visual box size=0.023 0.024 0.012

File: urdf/knolling_box/box_2.urdf (robot description, URDF)
Before this commit: robot 2x2, 1 links, 0 joints
Links:
- link base_link: geometry collision box size=0.021 0.026 0.012; visual box size=0.021 0.026 0.012

File: urdf/knolling_box/box_3.urdf (robot description, URDF)
Before this commit: robot 2x2, 1 links, 0 joints
Links:
- link base_link: geometry collision box size=0.035 0.038 0.012; visual box size=0.035 0.038 0.012

File: urdf/knolling_box/box_4.urdf (robot description, URDF)
Before this commit: robot 2x2, 1 links, 0 joints
Links:
- link base_link: geometry collision box size=0.025 0.029 0.012; visual box size=0.025 0.029 0.012

File: urdf/knolling_box/box_5.urdf (robot description, URDF)
Before this commit: robot 2x2, 1 links, 0 joints
Links:
- link base_link: geometry collision box size=0.026 0.029 0.012; visual box size=0.026 0.029 0.012

File: urdf/knolling_box/box_6.urdf (robot description, URDF)
Before this commit: robot 2x2, 1 links, 0 joints
Links:
- link base_link: geometry collision box size=0.02 0.028 0.012; visual box size=0.02 0.028 0.012

File: urdf/knolling_box/box_7.urdf (robot description, URDF)
Before this commit: robot 2x2, 1 links, 0 joints
Links:
- link base_link: geometry collision box size=0.022 0.028 0.012; visual box size=0.022 0.028 0.012

File: urdf/knolling_box/box_8.urdf (robot description, URDF)
Before this commit: robot 2x2, 1 links, 0 joints
Links:
- link base_link: geometry collision box size=0.03 0.045 0.012; visual box size=0.03 0.045 0.012

File: urdf/knolling_box/box_9.urdf (robot description, URDF)
Before this commit: robot 2x2, 1 links, 0 joints
Links:
- link base_link: geometry collision box size=0.02 0.02 0.012; visual box size=0.02 0.02 0.012

Commit message: zzz xps update

File: urdf/knolling_box/box_0.urdf (robot description, URDF)
Before this commit: robot 2x2, 1 links, 0 joints
Links:
- link base_link: geometry collision box size=0.037 0.027 0.012; visual box size=0.037 0.027 0.012

File: urdf/knolling_box/box_1.urdf (robot description, URDF)
Before this commit: robot 2x2, 1 links, 0 joints
Links:
- link base_link: geometry collision box size=0.034 0.03 0.012; visual box size=0.034 0.03 0.012

File: urdf/knolling_box/box_2.urdf (robot description, URDF)
Before this commit: robot 2x2, 1 links, 0 joints
Links:
- link base_link: geometry collision box size=0.019 0.025 0.012; visual box size=0.019 0.025 0.012

File: urdf/knolling_box/box_3.urdf (robot description, URDF)
Before this commit: robot 2x2, 1 links, 0 joints
Links:
- link base_link: geometry collision box size=0.025 0.029 0.012; visual box size=0.025 0.029 0.012

File: urdf/knolling_box/box_4.urdf (robot description, URDF)
Before this commit: robot 2x2, 1 links, 0 joints
Links:
- link base_link: geometry collision box size=0.021 0.021 0.012; visual box size=0.021 0.021 0.012

File: urdf/knolling_box/box_5.urdf (robot description, URDF)
Before this commit: robot 2x2, 1 links, 0 joints
Links:
- link base_link: geometry collision box size=0.035 0.025 0.012; visual box size=0.035 0.025 0.012

File: urdf/knolling_box/box_6.urdf (robot description, URDF)
Before this commit: robot 2x2, 1 links, 0 joints
Links:
- link base_link: geometry collision box size=0.025 0.027 0.012; visual box size=0.025 0.027 0.012

File: urdf/knolling_box/box_7.urdf (robot description, URDF)
Before this commit: robot 2x2, 1 links, 0 joints
Links:
- link base_link: geometry collision box size=0.04 0.02 0.012; visual box size=0.04 0.02 0.012

File: urdf/knolling_box/box_8.urdf (robot description, URDF)
Before this commit: robot 2x2, 1 links, 0 joints
Links:
- link base_link: geometry collision box size=0.019 0.034 0.012; visual box size=0.019 0.034 0.012

File: urdf/knolling_box/box_9.urdf (robot description, URDF)
Before this commit: robot 2x2, 1 links, 0 joints
Links:
- link base_link: geometry collision box size=0.019 0.026 0.012; visual box size=0.019 0.026 0.012

Commit message: Aug. 15

File: urdf/knolling_box/box_0.urdf (robot description, URDF)
Before this commit: robot 2x2, 1 links, 0 joints
Links:
- link base_link: geometry collision box size=0.021 0.023 0.012; visual box size=0.021 0.023 0.012

File: urdf/knolling_box/box_1.urdf (robot description, URDF)
Before this commit: robot 2x2, 1 links, 0 joints
Links:
- link base_link: geometry collision box size=0.018 0.02 0.012; visual box size=0.018 0.02 0.012

File: urdf/knolling_box/box_2.urdf (robot description, URDF)
Before this commit: robot 2x2, 1 links, 0 joints
Links:
- link base_link: geometry collision box size=0.035 0.029 0.012; visual box size=0.035 0.029 0.012

File: urdf/knolling_box/box_3.urdf (robot description, URDF)
Before this commit: robot 2x2, 1 links, 0 joints
Links:
- link base_link: geometry collision box size=0.017 0.038 0.012; visual box size=0.017 0.038 0.012

File: urdf/knolling_box/box_4.urdf (robot description, URDF)
Before this commit: robot 2x2, 1 links, 0 joints
Links:
- link base_link: geometry collision box size=0.026 0.027 0.012; visual box size=0.026 0.027 0.012

File: urdf/knolling_box/box_5.urdf (robot description, URDF)
Before this commit: robot 2x2, 1 links, 0 joints
Links:
- link base_link: geometry collision box size=0.031 0.025 0.012; visual box size=0.031 0.025 0.012

File: urdf/knolling_box/box_6.urdf (robot description, URDF)
Before this commit: robot 2x2, 1 links, 0 joints
Links:
- link base_link: geometry collision box size=0.029 0.027 0.012; visual box size=0.029 0.027 0.012

File: urdf/knolling_box/box_7.urdf (robot description, URDF)
Before this commit: robot 2x2, 1 links, 0 joints
Links:
- link base_link: geometry collision box size=0.025 0.025 0.012; visual box size=0.025 0.025 0.012

File: urdf/knolling_box/box_8.urdf (robot description, URDF)
Before this commit: robot 2x2, 1 links, 0 joints
Links:
- link base_link: geometry collision box size=0.04 0.031 0.012; visual box size=0.04 0.031 0.012

File: urdf/knolling_box/box_9.urdf (robot description, URDF)
Before this commit: robot 2x2, 1 links, 0 joints
Links:
- link base_link: geometry collision box size=0.017 0.018 0.012; visual box size=0.017 0.018 0.012
